File: Analog_IO_DC_Motor_LCD/ED/ED.kicad_sch (KiCad schematic)
At the start: 11 parts, among them M1 Motor_DC, SW1 SW_Push, SW2 SW_Push, U1 RC1602A, U2 L293D

Commit message: message in scheme
Other:
- note added: "(Optional capacitors)"
Changed lines of the file:
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@@
+		)
+	)
+	(text "(Optional capacitors)"
+		(exclude_from_sim no)
+		(at 44.196 82.296 0)
+		(effects
+			(font
+				(size 1.27 1.27)
+			)
 		)
 	)

Commit message: resistors and capacitors values into kicad project
Parts:
- 104_C1: renamed from C1; value C -> 0,1uF
- 104_C2: renamed from C2; value C -> 0,1uF
- R1, R2: value R -> 10kΩ
- RV1: value R_Potentiometer -> 10kΩ_Potentiometer
Changed lines of the file:
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@@
 		(dnp no)
 		(fields_autoplaced yes)
-		(property "Reference" "C1"
+		(property "Reference" "104_C1"
 			(at 46.99 73.6599 0)
 			(effects
@@
 			)
 		)
-		(property "Value" "C"
+		(property "Value" "0,1uF"
 			(at 46.99 76.1999 0)
 			(effects
@@
 			(project ""
 				(path "/012f2440-9ac9-45fd-9249-9d6bd5e615fe"
-					(reference "C1")
+					(reference "104_C1")
 					(unit 1)
 				)
@@
 			)
 		)
-		(property "Value" "R"
+		(property "Value" "10kΩ"
 			(at 38.1 76.1999 0)
 			(effects
@@
 			)
 		)
-		(property "Value" "R"
+		(property "Value" "10kΩ"
 			(at 38.1 91.4399 0)
 			(effects
@@
 		(dnp no)
 		(fields_autoplaced yes)
-		(property "Reference" "C2"
+		(property "Reference" "104_C2"
 			(at 46.99 88.8999 0)
 			(effects
@@
 			)
 		)
-		(property "Value" "C"
+		(property "Value" "0,1uF"
 			(at 46.99 91.4399 0)
 			(effects
@@
 			(project ""
 				(path "/012f2440-9ac9-45fd-9249-9d6bd5e615fe"
-					(reference "C2")
+					(reference "104_C2")
 					(unit 1)
 				)
@@
 			)
 		)
-		(property "Value" "R_Potentiometer"
+		(property "Value" "10kΩ_Potentiometer"
 			(at 128.27 58.4201 0)
 			(effects
@@
 			)
 		)
-		(property "Datasheet" "~"
+		(property "Datasheet" ""
 			(at 125.73 59.69 0)
 			(effects
